File: Board/EnergyMonitor.kicad_sch (KiCad schematic)
At the start: 56 parts, among them J2 RPi Zero, J3 Display, J4 Screw_Terminal_01x12, J5 Screw_Terminal_01x03, Q1 BSS138, Q2 BSS138, U1 MCP3424, U2 MCP3424, U3 WE-TVS-824014, U4 WE-TVS-824014

Commit message: fully routed pcb
Parts:
- C4, C6: footprint (none) -> Capacitor_Tantalum_SMD:CP_EIA-3216-18_Kemet-A_Pad1.58x1.35mm_HandSolder
- C8: footprint (none) -> Capacitor_SMD:CP_Elec_5x5.4
- J5: value Screw_Terminal_01x03 -> (none)
- JP3: value (none) -> VDDA Select
Other:
- moved on the sheet: C2, C3, C8, F1, J5, L1, PS1, RV1

Commit message: resized PCB slightly for a better fit in the case
Parts:
- F1: value 500mA -> (none); footprint Fuse:Fuseholder_Cylinder-5x20mm_Schurter_0031_8201_Horizontal_Open -> (none); Conrad 533467 - 62 -> 533467
- J5: value (none) -> AC In
- R3, R4: value 470k -> (none)
- U3, U4: value WE-TVS-824014 -> (none); footprint Package_TO_SOT_SMD:SOT-23-6 -> (none); Conrad (none) -> 1680500
Changed lines of the file:
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@@
       (effects (font (size 1.27 1.27)) (justify right))
     )
-    (property "Value" "WE-TVS-824014" (id 1) (at 244.475 134.62 0)
-      (effects (font (size 1.27 1.27)) (justify right))
-    )
-    (property "Footprint" "Package_TO_SOT_SMD:SOT-23-6" (id 2) (at 258.445 140.335 0)
+    (property "Value" "" (id 1) (at 244.475 134.62 0)
+      (effects (font (size 1.27 1.27)) (justify right))
+    )
+    (property "Footprint" "" (id 2) (at 258.445 140.335 0)
       (effects (font (size 1.27 1.27)) hide)
     )
     (property "Datasheet" "https://asset.conrad.com/media10/add/160267/c1/-/en/001680500DS01/datenblatt-1680500-wuerth-elektronik-tvs-diode-we-tvs-824014-sot-23-6l-6-v.pdf" (id 3) (at 260.985 140.335 0)
+      (effects (font (size 1.27 1.27)) hide)
+    )
+    (property "Conrad" "1680500" (id 4) (at 251.46 140.335 90)
       (effects (font (size 1.27 1.27)) hide)
     )
@@
     (in_bom yes) (on_board yes) (fields_autoplaced)
     (property "Reference" "J5" (id 0) (at 22.86 21.59 0))
-    (property "Value" "" (id 1) (at 22.86 24.13 0))
+    (property "Value" "AC In" (id 1) (at 22.86 24.13 0))
     (property "Footprint" "TerminalBlock_MetzConnect:TerminalBlock_MetzConnect_Type175_RT02703HBLC_1x03_P7.50mm_Horizontal" (id 2) (at 22.86 31.115 0)
       (effects (font (size 1.27 1.27)) hide)
@@
     (in_bom yes) (on_board yes) (fields_autoplaced)
     (property "Reference" "F1" (id 0) (at 38.735 29.21 90))
-    (property "Value" "500mA" (id 1) (at 38.735 31.75 90))
-    (property "Footprint" "Fuse:Fuseholder_Cylinder-5x20mm_Schurter_0031_8201_Horizontal_Open" (id 2) (at 38.735 36.703 90)
+    (property "Value" "" (id 1) (at 38.735 31.75 90))
+    (property "Footprint" "" (id 2) (at 38.735 36.703 90)
       (effects (font (size 1.27 1.27)) hide)
     )
@@
       (effects (font (size 1.27 1.27)) hide)
     )
-    (property "Conrad" "533467 - 62" (id 4) (at 38.735 34.925 90)
+    (property "Conrad" "533467" (id 4) (at 38.735 34.925 90)
       (effects (font (size 1.27 1.27)) hide)
     )
@@
       (effects (font (size 1.27 1.27)) (justify left))
     )
-    (property "Value" "470k" (id 1) (at 68.58 93.98 0)
+    (property "Value" "" (id 1) (at 68.58 93.98 0)
       (effects (font (size 1.27 1.27)) (justify left))
     )
@@
       (effects (font (size 1.27 1.27)) hide)
     )
-    (property "Value" "" (id 1) (at 40.132 20.32 90)
+    (property "Value" "SYM_Flash_Large" (id 1) (at 40.132 20.32 90)
       (effects (font (size 1.27 1.27)) hide)
     )
@@
       (effects (font (size 1.27 1.27)) (justify right))
     )
-    (property "Value" "WE-TVS-824014" (id 1) (at 258.445 134.62 0)
-      (effects (font (size 1.27 1.27)) (justify right))
-    )
-    (property "Footprint" "Package_TO_SOT_SMD:SOT-23-6" (id 2) (at 272.415 140.335 0)
+    (property "Value" "" (id 1) (at 258.445 134.62 0)
+      (effects (font (size 1.27 1.27)) (justify right))
+    )
+    (property "Footprint" "" (id 2) (at 272.415 140.335 0)
       (effects (font (size 1.27 1.27)) hide)
     )
     (property "Datasheet" "https://asset.conrad.com/media10/add/160267/c1/-/en/001680500DS01/datenblatt-1680500-wuerth-elektronik-tvs-diode-we-tvs-824014-sot-23-6l-6-v.pdf" (id 3) (at 274.955 140.335 0)
+      (effects (font (size 1.27 1.27)) hide)
+    )
+    (property "Conrad" "1680500" (id 4) (at 265.43 140.335 90)
       (effects (font (size 1.27 1.27)) hide)
     )
@@
       (effects (font (size 1.27 1.27)) (justify left))
     )
-    (property "Value" "470k" (id 1) (at 68.58 99.06 0)
+    (property "Value" "" (id 1) (at 68.58 99.06 0)
       (effects (font (size 1.27 1.27)) (justify left))
     )
@@
     )
     (path "/7eab9a7a-fd09-439e-8a57-83e9bd802247"
-      (reference "R3") (unit 1) (value "470k") (footprint "Resistor_SMD:R_1206_3216Metric_Pad1.30x1.75mm_HandSolder")
+      (reference "R3") (unit 1) (value "100k") (footprint "Resistor_SMD:R_1206_3216Metric_Pad1.30x1.75mm_HandSolder")
     )
     (path "/d1373e4c-a9af-4baa-ae56-bd386b97bef2"
-      (reference "R4") (unit 1) (value "470k") (footprint "Resistor_SMD:R_1206_3216Metric_Pad1.30x1.75mm_HandSolder")
+      (reference "R4") (unit 1) (value "100k") (footprint "Resistor_SMD:R_1206_3216Metric_Pad1.30x1.75mm_HandSolder")
     )
     (path "/84dc7d55-89e3-42fb-ab4c-cb0d709735ca"

Commit message: fixed some board layout issues after prototype assembly
Parts:
- F1: value (none) -> 500mA; footprint (none) -> Fuse:Fuseholder_Cylinder-5x20mm_Schurter_0031_8201_Horizontal_Open
- R3, R4: value (none) -> 100k
- U3, U4: value (none) -> WE-TVS-824014; footprint (none) -> Package_TO_SOT_SMD:SOT-23-6
Connections:
- net +5V: now also C3.1, C8.1; no longer C3.2, C8.2
- net GND: now also C3.2, C8.2; no longer C3.1, C8.1
- net LINE: now also L1.2; no longer L1.3
- net NEUT: now also L1.1; no longer L1.4
- net at C2.1, J5.3 (Pin_3), RV1.2: now also L1.3; no longer L1.2
- net at C2.2, F1.2, RV1.1: now also L1.4; no longer L1.1
Other:
- moved on the sheet: C3, C8, L1

Commit message: do not populate pull up resistor on Vrms line
Parts:
- R3: value 100k -> (none)
Changed lines of the file:
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@@
       (effects (font (size 1.27 1.27)) (justify left))
     )
-    (property "Value" "100k" (id 1) (at 68.58 93.98 0)
+    (property "Value" "" (id 1) (at 68.58 93.98 0)
       (effects (font (size 1.27 1.27)) (justify left))
     )
@@
     )
     (path "/7eab9a7a-fd09-439e-8a57-83e9bd802247"
-      (reference "R3") (unit 1) (value "100k") (footprint "Resistor_SMD:R_1206_3216Metric_Pad1.30x1.75mm_HandSolder")
+      (reference "R3") (unit 1) (value "DNP") (footprint "Resistor_SMD:R_1206_3216Metric_Pad1.30x1.75mm_HandSolder")
     )
     (path "/d1373e4c-a9af-4baa-ae56-bd386b97bef2"

Commit message: fixed offset voltage for vrms measurment
Parts:
- D1: value 5V -> (none)
- R4: value 100k -> (none)
Changed lines of the file:
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@@
       (effects (font (size 1.27 1.27)) (justify left))
     )
-    (property "Value" "5V" (id 1) (at 76.835 86.3599 90)
+    (property "Value" "" (id 1) (at 76.835 86.3599 90)
       (effects (font (size 1.27 1.27)) (justify left))
     )
@@
       (effects (font (size 1.27 1.27)) (justify left))
     )
-    (property "Value" "100k" (id 1) (at 68.58 99.06 0)
+    (property "Value" "" (id 1) (at 68.58 99.06 0)
       (effects (font (size 1.27 1.27)) (justify left))
     )
@@
     )
     (path "/96c91572-776f-407b-b536-76eeea4bf80e"
-      (reference "D1") (unit 1) (value "5V") (footprint "Diode_SMD:D_MiniMELF_Handsoldering")
+      (reference "D1") (unit 1) (value "DNP") (footprint "Diode_SMD:D_MiniMELF_Handsoldering")
     )
     (path "/36ca380b-9e35-4164-b404-4d5dc1ed6963"
@@
     )
     (path "/d1373e4c-a9af-4baa-ae56-bd386b97bef2"
-      (reference "R4") (unit 1) (value "100k") (footprint "Resistor_SMD:R_1206_3216Metric_Pad1.30x1.75mm_HandSolder")
+      (reference "R4") (unit 1) (value "10") (footprint "Resistor_SMD:R_1206_3216Metric_Pad1.30x1.75mm_HandSolder")
     )
     (path "/84dc7d55-89e3-42fb-ab4c-cb0d709735ca"
